Commit message: Updated lasers

File: segbot_description/robots/segbot_hokuyo.urdf.xacro (robot description, xacro)
@@ -14,6 +14,6 @@
   </xacro:segbot_chassis>
   <!-- Add the hokuyo -->
-  <xacro:hokuyo_mount name="nav_hokuyo" parent="front_left_vertical_beam" length="${SENSOR_BEAM_LENGTH*INCH_TO_M}" ros_topic="scan" update_rate="10" min_angle="${-(5 * M_PI)/12}" max_angle="${(5 * M_PI)/12}">
-    <origin xyz="0 -${0.5*INCH_TO_M} ${7*INCH_TO_M}" rpy="${M_PI/2} ${M_PI/2} 0" />
+  <xacro:hokuyo_mount name="nav_hokuyo" parent="front_right_vertical_beam" length="${SENSOR_BEAM_LENGTH*INCH_TO_M}" ros_topic="scan" update_rate="10" min_angle="${-(5 * M_PI)/12}" max_angle="${(5 * M_PI)/12}">
+    <origin xyz="0 ${0.5*INCH_TO_M} ${7*INCH_TO_M}" rpy="-${M_PI/2} -${M_PI/2} 0" />
   </xacro:hokuyo_mount>
   <xacro:gazebo_segbot_ros_controllers />

File: segbot_description/robots/segbot_navigation.urdf.xacro (robot description, xacro)
@@ -19,6 +19,6 @@
   </xacro:kinect_mount>
   <!-- Add the hokuyo -->
-  <xacro:hokuyo_mount name="nav_hokuyo" parent="front_left_vertical_beam" length="${SENSOR_BEAM_LENGTH*INCH_TO_M}" ros_topic="scan" update_rate="10" min_angle="${-(5 * M_PI)/12}" max_angle="${(5 * M_PI)/12}">
-    <origin xyz="0 -${0.5*INCH_TO_M} ${7*INCH_TO_M}" rpy="${M_PI/2} ${M_PI/2} 0" />
+  <xacro:hokuyo_mount name="nav_hokuyo" parent="front_right_vertical_beam" length="${SENSOR_BEAM_LENGTH*INCH_TO_M}" ros_topic="scan" update_rate="10" min_angle="${-(5 * M_PI)/12}" max_angle="${(5 * M_PI)/12}">
+    <origin xyz="0 ${0.5*INCH_TO_M} ${7*INCH_TO_M}" rpy="-${M_PI/2} -${M_PI/2} 0" />
   </xacro:hokuyo_mount>
   <xacro:gazebo_segbot_ros_controllers />

File: segbot_description/urdf/sensors/hokuyo_04lx_laser.gazebo.xacro (robot description, xacro)
@@ -20,5 +20,5 @@
           <range>
             <min>0.02</min>
-            <max>4.0</max>
+            <max>20.0</max>
             <resolution>0.03</resolution>
           </range>
